File: Buck_Converter_Altium_to_KiCAD/Buck_Conveter_PCB.kicad_sch (KiCad schematic)
At the start: 20 parts, among them J1 XT30, J2 XT30, U1 LM61495RPHR

Commit message: Updated pcb with LED
Parts:
- added D1: LED Indicator, 2V_LED, symbol Buck_Conveter_PCB-altium-import:root_3_150060VS75000
- added R1: 100K, 100k Resistor, symbol Buck_Conveter_PCB-altium-import:root_1_CRCW0402100KFKED
Connections:
- net 5V_OUT: now also R1.2
- net GND: now also D1.2 (A)
- new net: D1.1 (K), R1.1

Commit message: Updated PCB
Parts:
- removed CBoot1: 100nF, Cboot_100nF, symbol Buck_Conveter_PCB-altium-import:root_1_GRM155R71A104KA01D
- removed CFF1: 5.1pF, CFF_5.1pf, symbol Buck_Conveter_PCB-altium-import:root_1_GRM1555C1E5R1CA01D
- removed Cbias1: 100nF, Cbias_100nF, symbol Buck_Conveter_PCB-altium-import:root_1_GRM155R71C104KA88D
- removed R1, Rfbt: 100K, 100k Resistor, symbol Buck_Conveter_PCB-altium-import:root_1_CRCW0402100KFKED
- removed Rfbb: 24.9K, R_Fbb_24.9k, symbol Buck_Conveter_PCB-altium-import:root_1_RC0603FR-0724K9L
- removed Rff: 4.99K, 4.99K_Resistor, symbol Buck_Conveter_PCB-altium-import:root_0_CRCW04024K99FKED
- removed Rreset: 100K, 100k Resistor, symbol Buck_Conveter_PCB-altium-import:root_0_CRCW0402100KFKED
- added CBoot1, Cbias1: 100nF, Cboot_100nF, symbol Buck_Conveter_PCB-altium-import:root_1_CC0603KRX7R7BB104
- added CFF1: 5.1pF, CFF_5.1pf, symbol Buck_Conveter_PCB-altium-import:root_1_CC0603CRNPO9BN5R1
- added R1, Rfbt: 100k, 100k Resistor, symbol Buck_Conveter_PCB-altium-import:root_1_RMCF0603FT100K
- added R2: 50, 50_Resistor, symbol Buck_Conveter_PCB-altium-import:root_3_CRCW060350R0FKEA
- added Rfbb: 24.9k, R_Fbb_24.9k, symbol Buck_Conveter_PCB-altium-import:root_1_CRCW060324K9FKEA
- added Rff: 4.99K, 4.99K_Resistor, symbol Buck_Conveter_PCB-altium-import:root_0_ERJ-3EKF4991V
- added Rreset: 100k, 100k Resistor, symbol Buck_Conveter_PCB-altium-import:root_0_RMCF0603FT100K
Connections:
- net 5V_OUT: now also CFF1.2, Cbias1.2, R1.2, Rfbt.2, Rreset.2
- net FB_IN: now also R2.2, Rfbb.2, Rff.1
- net GND: now also Cbias1.1, Rfbb.1
- net at U1.10 (RESET): now also Rreset.1
- net at D1.1 (K): now also R1.1
- net at L1.1, U1.16 (SW): now also CBoot1.2
- net at U1.3 (RBOOT), U1.4 (CBOOT): now also CBoot1.1
- new net: CFF1.1, Rff.2
- new net: R2.1, Rfbt.1
