File: Buck_Converter_Altium_to_KiCAD/Buck_Conveter_PCB.kicad_pcb (KiCad board)
At the start: 4 copper layers, 101.6 x 50.8 mm, 20 parts, among them J1 XT30, J2 XT30, U1 LM61495RPHR

Commit message: Updated pcb with LED
Parts:
- added D1: LED Indicator, Buck_PCB_Lib.PcbLib:2V_LED, F.Cu at (162.4, 119.7)
- added R1: 100K, Buck_PCB_Lib.PcbLib:100k Resistor, F.Cu at (158.3, 119.7)
Routing:
- net 5V_OUT: track 82.8 -> 89.5 mm
- net NetD1_1: track 0.00 -> 2.70 mm

Commit message: Updated PCB
Parts:
- removed CBoot1: 100nF, Buck_PCB_Lib.PcbLib:CBOOT_100NF
- removed Cbias1: 100nF, Buck_PCB_Lib.PcbLib:CBIAS_100NF
- removed CinHF1: 1uF, Buck_PCB_Lib.PcbLib:1UF_CINHF
- added CBoot: 100nF, Buck_PCB_Lib.PcbLib:CBOOT_100NF, F.Cu at (135.6, 101.0)
- added Cbias: 100nF, Buck_PCB_Lib.PcbLib:CBOOT_100NF, F.Cu at (131.6, 100.2)
- added Cin_HF1: 1uF, Buck_PCB_Lib.PcbLib:1UF_CINHF, F.Cu at (139.6, 101.3)
- added R2: 50, Buck_PCB_Lib.PcbLib:50_RESISTOR, F.Cu at (126.5, 104.5)
- R1: footprint Buck_PCB_Lib.PcbLib:100k Resistor -> Buck_PCB_Lib.PcbLib:100K RESISTOR
- moved Rfbt 4.65 mm to (124.1, 104.8), turned to 90 degrees
- moved CFF1 3.67 mm to (125.2, 100.1)
- moved Rff 2.57 mm to (128.4, 100.7)
- moved Cin1 1.80 mm to (140.1, 97.0), turned to -90 degrees
- moved Rfbb 1.39 mm to (129.1, 104.4), turned to 90 degrees
- moved Cin2 1.00 mm to (139.0, 111.3)
- moved Rreset 0.89 mm to (132.6, 108.0), turned to 180 degrees
- moved Cin_HF2 0.75 mm to (138.1, 108.0)
- moved Cout3 0.75 mm to (153.9, 95.6)
- moved Cout4 0.75 mm to (159.7, 95.6)
- moved Cvcc1 0.75 mm to (131.7, 104.3)
- moved U1 0.75 mm to (136.4, 104.9)
- moved R1 0.51 mm to (158.4, 120.2), turned to 180 degrees
- moved Cout1 0.50 mm to (153.9, 114.3)
- moved Cout2 0.50 mm to (159.7, 114.3)
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Connections:
- net Net'_1 renamed NetRreset_1
- Rfbt pad 1: FB_IN -> NetR2_1
Routing:
- net FB_IN: track 7.48 -> 10.6 mm
- net 12V_IN: track 0.00 -> 2.91 mm
- net NetR2_1: track 0.00 -> 2.44 mm
- net 5V_OUT: track 89.5 -> 91.6 mm
- net NetCboot1_2: track 11.9 -> 13.3 mm
- net NetCFF1_1: track 1.42 -> 2.45 mm
- net NetCboot1_1: track 2.13 -> 3.08 mm
- net VCC: track 9.74 -> 10.3 mm
- added copper zone on B.Cu, net GND
Other:
- board text added: "Vin"
- board text added: "Vout"

Commit message: Updated PCB
Other:
- board text added: "5V"
